Commit message: urdfとナビゲーションパラメータのチューニング

File: urdf/midori_cart.urdf (robot description, URDF)
Before this commit: robot midori_cart, 7 links, 6 joints
Links:
- link base_link: geometry collision box size=0.520 0.520 0.5
- link wheel_left_link: geometry collision cylinder length=0.06 radius=0.105
- link wheel_right_link: geometry collision cylinder length=0.06 radius=0.105
Joints:
- joint base_joint: origin xyz=0.0 0.0 0.010 rpy=0 0 0 -> xyz=0.0 0.0 0.1 rpy=0 0 0
- joint wheel_left_joint: origin xyz=0.0 0.08 0.023 rpy=-1.57 0 0 -> xyz=0.0 0.27 0.0 rpy=-1.57 0 0
- joint wheel_right_joint: origin xyz=0.0 -0.080 0.023 rpy=-1.57 0 0 -> xyz=0.0 -0.27 0.0 rpy=-1.57 0 0
